File: gaia-filler.kicad_pcb (KiCad board)
At the start: 2 copper layers, 50 x 50 mm, 2 parts, among them J2 Conn_02x10_Odd_Even, J3 Conn_02x10_Odd_Even

Commit message: filler routing+prod files
Connections:
- J2 pad 1: I2C_2_SDA -> unconnected-(J2-Pin_1-Pad1)
- J2 pad 2: I2C_1_SDA -> unconnected-(J2-Pin_2-Pad2)
- J2 pad 3: I2C_2_SCL -> unconnected-(J2-Pin_3-Pad3)
- J2 pad 4: I2C_1_SCL -> unconnected-(J2-Pin_4-Pad4)
Other:
- outline, holes or cut-outs redrawn
